File: Hardware/BusinessSynth/BusinessSynth.kicad_pcb (KiCad board)
At the start: 2 copper layers, 96 x 55 mm, 63 parts, among them J1 StylusKey, J2 StylusKey, J3 StylusKey, J4 StylusKey, J5 StylusKey, J6 StylusKey, J7 StylusKey, J8 StylusKey, J9 StylusKey, U1 ATtiny817-M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

Commit message: Finalize PCB for rev 2
Parts:
- added H3: Strain relief, MountingHole:MountingHole_2.1mm, F.Cu at (193.5, 72.2)
- added REF**: MountingHole_2mm, MountingHole:MountingHole_2mm, F.Cu at (190.5, 112.0)
- added REF**: MountingHole_2mm, MountingHole:MountingHole_2mm, F.Cu at (190.5, 113.0)
- added REF**: MountingHole_2mm, MountingHole:MountingHole_2mm, F.Cu at (190.5, 114.0)
- added REF**: MountingHole_2mm, MountingHole:MountingHole_2mm, F.Cu at (190.5, 88.0)
- added REF**: MountingHole_2mm, MountingHole:MountingHole_2mm, F.Cu at (190.5, 90.0)
- added REF**: MountingHole_2mm, MountingHole:MountingHole_2mm, F.Cu at (190.5, 89.0)
- H1, H2: footprint Connector_Wire:SolderWirePad_1x01_Drill0.8mm -> Connector_PinHeader_2.54mm:PinHeader_1x01_P2.54mm_Vertical
- J1: value StylusKey -> UPDI; footprint BusinessSynth:StylusKey -> Connector_PinHeader_2.54mm:PinHeader_1x03_P2.54mm_Vertical
- moved J1 3.46 mm to (187.4, 105.4), turned to 180 degrees
- moved H1 2.25 mm to (193.5, 74.5)
- moved R26 1.10 mm to (174.0, 97.6)
- moved R33 1.00 mm to (176.5, 102.5)
- moved R27 0.80 mm to (176.5, 98.3)
- moved R32 0.70 mm to (174.0, 101.8)
- moved R28 0.50 mm to (174.0, 99.0)
- moved R31 0.40 mm to (176.5, 101.1)
- moved R29 0.20 mm to (176.5, 99.7)
- moved R30 0.10 mm to (174.0, 100.4)
- turned LS1 to 206.6 degrees
- turned LS2 to 26.6 degrees
Connections:
- J1 pad 1: Net-(J1-Pad1) -> VDD
- U1 pad 23: Net-(J1-Pad1) -> Net-(J1-Pad3)
Routing:
- net /StylusGND: track 0.00 -> 48.5 mm
- net Net-(J1-Pad3): track 0.00 -> 6.38 mm, vias 0 -> 1
- net Net-(D8-Pad1): track 74.0 -> 76.9 mm
- net Net-(LS1-Pad2): track 10.5 -> 13.3 mm
- net Net-(R31-Pad1): track 6.76 -> 8.94 mm
- net Net-(J1-Pad1): track 1.21 -> 0.00 mm, vias 1 -> 0
- net Net-(D1-Pad1): track 16.8 -> 18.0 mm
- net Net-(C2-Pad1): track 18.1 -> 19.2 mm
- net Net-(LS1-Pad1): track 6.19 -> 7.29 mm
- net /KeyC3: track 28.4 -> 27.4 mm
- net Net-(D7-Pad1): track 78.1 -> 79.0 mm
- net Net-(D2-Pad1): track 19.3 -> 20.0 mm
Other:
- board text added: "Snap off"
- board text added: "pitch"
- board text added: "sondreixix@gmail.com github.com/sondre99v +47 464 21 647"
- board text removed: "+47 464 21 647 sondreixix@gmail.com github.com/sondre99v"
- board text removed: "mode"
- board text removed: "oct"
