File: Hardware/BusinessSynth/BusinessSynth.sch (KiCad schematic (older format))
At the start: 63 parts, among them J1 StylusKey, J2 StylusKey, J3 StylusKey, J4 StylusKey, J5 StylusKey, J6 StylusKey, J7 StylusKey, J8 StylusKey, J9 StylusKey, U1 ATtiny817-M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

Commit message: Finalize PCB for rev 2
Parts:
- removed J1: StylusKey, BusinessSynth:StylusKey, symbol BusinessSynth:StylusKey
- added J1: UPDI, Connector_PinHeader_2.54mm:PinHeader_1x03_P2.54mm_Vertical, symbol Connector:Conn_01x03_Female
Connections:
- wire segments 175 -> 179
Changed lines of the file:
@@
-	-1   0    0    -1
-$EndComp
-Wire Wire Line
-	4200 2350 4200 2150
-$Comp
-L BusinessSynth:StylusKey J1
-U 1 1 5CABA3B5
-P 4300 2150
-F 0 "J1" H 4172 2201 50  0000 R CNN
-F 1 "StylusKey" H 4172 2110 50  0000 R CNN
-F 2 "BusinessSynth:StylusKey" H 4200 2150 50  0001 C CNN
-F 3 "" H 4200 2150 50  0001 C CNN
-	1    4300 2150
 	-1   0    0    -1
 $EndComp
@@
 	1    0    0    -1
 $EndComp
+$Comp
+L Connector:Conn_01x03_Female J1
+U 1 1 5D8E9631
+P 4400 1800
+F 0 "J1" H 4428 1826 50  0000 L CNN
+F 1 "UPDI" H 4428 1735 50  0000 L CNN
+F 2 "Connector_PinHeader_2.54mm:PinHeader_1x03_P2.54mm_Vertical" H 4400 1800 50  0001 C CNN
+F 3 "~" H 4400 1800 50  0001 C CNN
+	1    4400 1800
+	1    0    0    -1
+$EndComp
+Wire Wire Line
+	4200 1900 4200 2350
+$Comp
+L power:GND #PWR?
+U 1 1 5D8F5E83
+P 4050 1850
+F 0 "#PWR?" H 4050 1600 50  0001 C CNN
+F 1 "GND" H 4055 1677 50  0000 C CNN
+F 2 "" H 4050 1850 50  0001 C CNN
+F 3 "" H 4050 1850 50  0001 C CNN
+	1    4050 1850
+	1    0    0    -1
+$EndComp
+$Comp
+L power:VDD #PWR?
+U 1 1 5D8F62AA
+P 4050 1650
+F 0 "#PWR?" H 4050 1500 50  0001 C CNN
+F 1 "VDD" H 4067 1823 50  0000 C CNN
+F 2 "" H 4050 1650 50  0001 C CNN
+F 3 "" H 4050 1650 50  0001 C CNN
+	1    4050 1650
+	1    0    0    -1
+$EndComp
+Wire Wire Line
+	4050 1650 4050 1700
+Wire Wire Line
+	4050 1700 4200 1700
+Wire Wire Line
+	4200 1800 4050 1800
+Wire Wire Line
+	4050 1800 4050 1850
 $EndSCHEMATC
